Commit message: Added stereo camera

File: rover_description/urdf/camera.urdf.xacro (robot description, xacro)
@@ -1,71 +1,66 @@
 <?xml version="1.0"?>
-<robot xmlns:xacro="http://www.ros.org/wiki/xacro" name="camera">
-<xacro:property name="pi" value="3.1415926535897931"/>
-<xacro:macro name="camera" params="name parent hfov image_width image_height xyz rpy">
-  <!-- Suggested values: hfov="1.3962634" image_width="800" image_height="800" -->
-  <link name="${name}_link">
-    <collision>
-      <origin xyz="0 0 0" rpy="0 0 0"/>
-      <geometry>
-          <box size="0.02 0.08 0.05"/>
-      </geometry>
-    </collision>
-    <visual>
-      <origin xyz="0 0 0" rpy="0 0 0"/>
-      <geometry>
-          <box size="0.02 0.08 0.05"/>
-      </geometry>
-    </visual>
-    <inertial>
-      <mass value="0.0001" />
-      <origin xyz="0 0 0" rpy="0 0 ${pi}"/>
-      <inertia ixx="0.0000001" ixy="0" ixz="0" iyy="0.0000001" iyz="0" izz="0.0000001" />
-    </inertial>
-  </link>
-  <joint name="${name}_joint" type="fixed">
-    <axis xyz="0 1 0" />
-    <origin xyz="${xyz}" rpy="${rpy}"/>
-    <parent link="${parent}"/>
-    <child link="${name}_link"/>
-  </joint>
-  <gazebo reference="${name}_link">
-    <sensor type="camera" name="camera1">
-      <update_rate>30.0</update_rate>
-      <camera name="head">
-        <horizontal_fov>1.3962634</horizontal_fov>
-        <image>
-          <width>800</width>
-          <height>800</height>
-          <format>R8G8B8</format>
-        </image>
-        <clip>
-          <near>0.02</near>
-          <far>300</far>
-        </clip>
-        <noise>
-          <type>gaussian</type>
-          <!-- Noise is sampled independently per pixel on each frame.
-               That pixel's noise value is added to each of its color
-               channels, which at that point lie in the range [0,1]. -->
-          <mean>0.0</mean>
-          <stddev>0.007</stddev>
-        </noise>
-      </camera>
-      <plugin name="camera_controller" filename="libgazebo_ros_camera.so">
-        <alwaysOn>true</alwaysOn>
-        <updateRate>0.0</updateRate>
-        <cameraName>rover/camera1</cameraName>
-        <imageTopicName>image_raw</imageTopicName>
-        <cameraInfoTopicName>camera_info</cameraInfoTopicName>
-        <frameName>camera1_link</frameName>
-        <hackBaseline>0.07</hackBaseline>
-        <distortionK1>0.0</distortionK1>
-        <distortionK2>0.0</distortionK2>
-        <distortionK3>0.0</distortionK3>
-        <distortionT1>0.0</distortionT1>
-        <distortionT2>0.0</distortionT2>
-      </plugin>
-    </sensor>
-  </gazebo>
-</xacro:macro>
+<robot xmlns:xacro="http://www.ros.org/wiki/xacro">
+    <xacro:macro name="camera_sensor" params="name parent hfov image_width image_height *origin">
+      <link name="${name}_link">
+        <collision>
+          <origin xyz="0 0 0" rpy="0 0 0"/>
+          <geometry>
+              <box size="0.02 0.08 0.05"/>
+          </geometry>
+        </collision>
+        <visual>
+          <origin xyz="0 0 0" rpy="0 0 0"/>
+          <geometry>
+              <box size="0.02 0.08 0.05"/>
+          </geometry>
+        </visual>
+        <inertial>
+          <mass value="0.0001" />
+          <origin xyz="0 0 0" rpy="0 0 ${pi}"/>
+          <inertia ixx="0.0000001" ixy="0" ixz="0" iyy="0.0000001" iyz="0" izz="0.0000001" />
+        </inertial>
+      </link>
+      <joint name="${name}_joint" type="fixed">
+        <axis xyz="0 0 1" />
+          <xacro:insert_block name="origin"/>
+        <parent link="${parent}"/>
+        <child link="${name}_link"/>
+      </joint>
+      <gazebo reference="${name}_link">
+        <sensor type="camera" name="${name}">
+          <update_rate>30.0</update_rate>
+          <camera name="${name}">
+            <horizontal_fov>${hfov}</horizontal_fov>
+            <image>
+              <width>${image_width}</width>
+              <height>${image_height}</height>
+              <format>R8G8B8</format>
+            </image>
+            <clip>
+              <near>0.02</near>
+              <far>300</far>
+            </clip>
+            <noise>
+              <type>gaussian</type>
+              <mean>0.0</mean>
+              <stddev>0.007</stddev>
+            </noise>
+          </camera>
+          <plugin name="camera_controller" filename="libgazebo_ros_camera.so">
+            <alwaysOn>true</alwaysOn>
+            <updateRate>0.0</updateRate>
+            <cameraName>$(arg robot_namespace)/${name}</cameraName>
+            <imageTopicName>image_raw</imageTopicName>
+            <cameraInfoTopicName>camera_info</cameraInfoTopicName>
+            <frameName>${name}_link</frameName>
+            <hackBaseline>0.07</hackBaseline>
+            <distortionK1>0.0</distortionK1>
+            <distortionK2>0.0</distortionK2>
+            <distortionK3>0.0</distortionK3>
+            <distortionT1>0.0</distortionT1>
+            <distortionT2>0.0</distortionT2>
+          </plugin>
+        </sensor>
+      </gazebo>
+    </xacro:macro>
 </robot>

File: rover_description/urdf/rover.urdf.xacro (robot description, xacro)
@@ -1,5 +1,6 @@
 <?xml version="1.0" ?>
 <robot name="rover" xmlns:xacro="http://ros.org/wiki/xacro">
-  <xacro:include filename="$(find rover_description)/urdf/camera_test.urdf.xacro"/>
+  <xacro:include filename="$(find rover_description)/urdf/camera.urdf.xacro"/>
+  <xacro:include filename="$(find rover_description)/urdf/stereo_camera.urdf.xacro"/>
   <xacro:arg name="robot_namespace" default="/" />
   <!-- TODO: adjust geometry-->
@@ -117,5 +118,11 @@
   </xacro:wheel>
   <!-- Camera -->
-  <xacro:camera_sensor name="camera1" xyz="0 0 1" hfov="1.3962634" image_width="800" image_height="600" rpy="0 0 0" parent="base_link" />
+  <xacro:camera_sensor name="camera1" parent="base_link" hfov="1.3962634" image_width="800" image_height="600"  >
+    <origin xyz="0 0 0.5" rpy="0 0 0" />
+  </xacro:camera_sensor>
+  <!-- Stereo camera -->
+  <xacro:stereo_camera_sensor name="stereo_camera" parent="base_link" hfov="1.3962634" image_width="800" image_height="600" camera_distance="0.1" >
+    <origin xyz="${base_x_size/2} 0 0" rpy="0 0 0" />
+  </xacro:stereo_camera_sensor>
   <!-- gazebo plugins -->
   <gazebo>

File: rover_description/urdf/stereo_camera.urdf.xacro (robot description, xacro)
@@ -1,55 +1,94 @@
 <?xml version="1.0"?>
 <robot xmlns:xacro="http://www.ros.org/wiki/xacro">
-  <!-- stereo camera macro uses wge100_camera macros -->
-  <!--<xacro:include filename="$(find pr2_description)/urdf/sensors/wge100_camera.urdf.xacro" />
-  <xacro:include filename="$(find pr2_description)/urdf/sensors/stereo_camera.gazebo.xacro" />-->
-  <xacro:property name="stereo_dx" value="0.00" />
-  <xacro:property name="stereo_dy" value="-0.09" /> <!-- +y to the left -->
-  <xacro:property name="stereo_dz" value="0.00" />
-  <xacro:property name="stereo_rx" value="0.00" />
-  <xacro:property name="stereo_ry" value="0.00" />
-  <xacro:property name="stereo_rz" value="0.00" />
-  <!-- this macro is used for creating wide and narrow double stereo camera links -->
-  <xacro:macro name="stereo_camera_v0" params="name parent focal_length hfov image_format image_width image_height *origin">
-    <joint name="${name}_frame_joint" type="fixed">
-      <xacro:insert_block name="origin" />
-      <parent link="${parent}"/>
-      <child link="${name}_link"/>
-    </joint>
-    <!-- camera link is at center of the optical frame, but in x-forward notation -->
-    <link name="${name}_link">
+  <xacro:include filename="$(find rover_description)/urdf/camera.urdf.xacro"/>
+  <xacro:macro name="stereo_camera_sensor" params="name parent hfov image_width image_height camera_distance *origin" >
+    <xacro:property name="frame_thickness" value="0.01" />
+    <link name="${name}_frame" >
+      <collision>
+        <origin xyz="${frame_thickness} 0 0" rpy="0 0 0"/>
+        <geometry>
+            <box size="${frame_thickness} ${camera_distance+0.08} 0.05"/>
+        </geometry>
+      </collision>
+      <visual>
+        <origin xyz="${frame_thickness} 0 0" rpy="0 0 0"/>
+        <geometry>
+            <box size="${frame_thickness} ${camera_distance+0.08} 0.05"/>
+        </geometry>
+      </visual>
       <inertial>
-        <mass value="0.1" />
-        <origin xyz="0 0 0" rpy="0 0 0" />
-        <inertia ixx="0.01"  ixy="0"  ixz="0" iyy="0.01"  iyz="0"  izz="0.01" /> <!-- this inertia is made up for now. -->
+        <mass value="0.0001" />
+        <origin xyz="${frame_thickness} 0 0" rpy="0 0 ${pi}"/>
+        <inertia ixx="0.0000001" ixy="0" ixz="0" iyy="0.0000001" iyz="0" izz="0.0000001" />
       </inertial>
     </link>
-    <!-- attach optical frame to the camera link -->
-    <joint name="${name}_optical_frame_joint" type="fixed">
-      <origin xyz="0 0 0" rpy="${-M_PI/2} 0.0 ${-M_PI/2}" /> <!-- rotate frame from x-forward to z-forward camera coords -->
-      <parent link="${name}_link"/>
+    <joint name="${name}_joint" type="fixed">
+      <axis xyz="0 1 0" />
+        <xacro:insert_block name="origin"/>
+      <parent link="${parent}"/>
+      <child link="${name}_frame"/>
+    </joint>
+    <link name="${name}_optical_frame" />
+    <joint name="${name}_optical_joint" type="fixed">
+      <axis xyz="0 1 0" />
+        <origin xyz="0 0 0" rpy="${-pi/2} 0 ${-pi/2}" />
+      <parent link="${name}_frame"/>
       <child link="${name}_optical_frame"/>
     </joint>
-    <!-- optical frame for the stereo camera, with z-forward notation, this is the frame stereo camera images users should refer to -->
-    <link name="${name}_optical_frame" type="camera"/>
-    <!-- stereo left camera -->
-    <xacro:wge100_camera_v0 name="${name}_l_stereo_camera" camera_name="${name}/left" image_format="${image_format}" image_topic_name="image_raw"
-                            camera_info_topic_name="camera_info" parent="${name}_link"
-                            hfov="${hfov}" focal_length="${focal_length}"
-                            frame_id="${name}_optical_frame" hack_baseline="0"
-                            image_width="${image_width}" image_height="${image_height}">
-      <origin xyz="0 0 0" rpy="0 0 0" />
-    </xacro:wge100_camera_v0>
-    <!-- stereo right camera -->
-    <xacro:wge100_camera_v0 name="${name}_r_stereo_camera" camera_name="${name}/right" image_format="${image_format}" image_topic_name="image_raw"
-                            camera_info_topic_name="camera_info" parent="${name}_l_stereo_camera_frame"
-                            hfov="${hfov}" focal_length="${focal_length}"
-                            frame_id="${name}_optical_frame" hack_baseline="${-stereo_dy}"
-                            image_width="${image_width}" image_height="${image_height}">
-      <origin xyz="${stereo_dx} ${stereo_dy} ${stereo_dz}" rpy="${stereo_rx} ${stereo_ry} ${stereo_rz}" />
-    </xacro:wge100_camera_v0>
-    <!-- extensions -->
-    <xacro:stereo_camera_gazebo_v0 name="${name}" focal_length="${focal_length}" hfov="${hfov}"
-                                   image_width="${image_width}" image_height="${image_height}"/>
+    <gazebo reference="${name}_frame">
+      <sensor type="multicamera" name="${name}">
+        <update_rate>30.0</update_rate>
+        <camera name="left">
+          <pose>${frame_thickness} ${camera_distance/2} 0 0 0 0</pose>
+          <horizontal_fov>${hfov}</horizontal_fov>
+          <image>
+            <width>${image_width}</width>
+            <height>${image_height}</height>
+            <format>R8G8B8</format>
+          </image>
+          <clip>
+            <near>0.02</near>
+            <far>300</far>
+          </clip>
+          <noise>
+            <type>gaussian</type>
+            <mean>0.0</mean>
+            <stddev>0.007</stddev>
+          </noise>
+        </camera>
+        <camera name="right">
+          <pose>${frame_thickness} ${-camera_distance/2} 0 0 0 0</pose>
+          <horizontal_fov>${hfov}</horizontal_fov>
+          <image>
+            <width>${image_width}</width>
+            <height>${image_height}</height>
+            <format>R8G8B8</format>
+          </image>
+          <clip>
+            <near>0.02</near>
+            <far>300</far>
+          </clip>
+          <noise>
+            <type>gaussian</type>
+            <mean>0.0</mean>
+            <stddev>0.007</stddev>
+          </noise>
+        </camera>
+        <plugin name="stereo_camera_controller" filename="libgazebo_ros_multicamera.so">
+          <alwaysOn>true</alwaysOn>
+          <updateRate>5.0</updateRate>
+          <cameraName>${name}</cameraName>
+          <imageTopicName>image_raw</imageTopicName>
+          <cameraInfoTopicName>camera_info</cameraInfoTopicName>
+          <frameName>${name}_optical_frame</frameName>
+          <hackBaseline>${camera_distance}</hackBaseline>
+          <distortionK1>0.0</distortionK1>
+          <distortionK2>0.0</distortionK2>
+          <distortionK3>0.0</distortionK3>
+          <distortionT1>0.0</distortionT1>
+          <distortionT2>0.0</distortionT2>
+        </plugin>
+      </sensor>
+    </gazebo>
   </xacro:macro>
 </robot>
